File: T5848.kicad_pcb (KiCad board)
At the start: 2 copper layers, 58.4 x 22.9 mm, 20 parts, among them J1 Conn_01x16_Pin, J2 Conn_01x12_Pin, J3 Conn_01x02, U2 TLV7A03_SOT23-5, U3 TXB0108DQSR

Commit message: updates
Parts:
- added REF**: LordsBoardsLogo_Small_Silk, LordsBoards-Symbol:LordsBoardsLogo_Medium_Silk, F.Cu at (145.3, 102.7)
Routing:
- net VDD: track 15.2 -> 59.3 mm, vias 1 -> 2
- net +1.8V: track 14.4 -> 50.0 mm, vias 2 -> 3
- net /SD: track 1.31 -> 29.2 mm
- net /SCK_{LS}: track 16.8 -> 43.8 mm, vias 1 -> 2
- net /THSEL_1: track 2.17 -> 28.7 mm
- net /WAKE_1: track 1.84 -> 24.8 mm
- net /SD_{LS}: track 9.93 -> 32.4 mm, vias 1 -> 2
- net /WS_{LS}: track 7.38 -> 29.4 mm, vias 1 -> 2
- net /WS: track 42.7 -> 46.3 mm, vias 0 -> 1
- net /SCK: track 43.5 -> 46.8 mm, vias 0 -> 1
- net /THSEL_1_{LS}: track 32.6 -> 35.4 mm
- net GND: track 16.8 -> 17.7 mm, vias 10 -> 19
- added copper zone on In1.Cu, net GND
- added copper zone on In2.Cu, net GND
Other:
- copper layers 2 -> 4
- board text added: "Dual T5848 Microphone FeatherWing"
- board text removed: "Dual T5848 Microphone Expansion Board"
